File: PCB/UserInterface/User Interface.brd (EAGLE design)
At the start: 66.1 x 53.3 mm, 25 parts

Commit message: update user interface
Parts:
- R1, R10, R11, R2, R3, R4, R5, R6, R7, R8, R9: value (none) -> 470
Changed lines of the file:
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@@
 <attribute name="SF_SKU" value="COM-00097" x="22.86" y="19.05" size="1.778" layer="27" display="off"/>
 </element>
-<element name="R1" library="SparkFun-Resistors" package="1206" value=" " x="44.45" y="48.26" smashed="yes" rot="MR270">
+<element name="R1" library="SparkFun-Resistors" package="1206" value="470" x="44.45" y="48.26" smashed="yes" rot="MR270">
 <attribute name="NAME" x="44.45" y="48.26" size="0.762" layer="22" font="vector" ratio="20" rot="MR0" align="center"/>
 <attribute name="PROD_ID" value=" " x="44.45" y="48.26" size="1.778" layer="28" rot="MR270" display="off"/>
 <attribute name="VALUE" x="45.593" y="48.26" size="0.6096" layer="28" font="vector" ratio="20" rot="MR270" align="top-center"/>
 </element>
-<element name="R10" library="SparkFun-Resistors" package="1206" value=" " x="21.59" y="48.26" smashed="yes" rot="MR270">
+<element name="R10" library="SparkFun-Resistors" package="1206" value="470" x="21.59" y="48.26" smashed="yes" rot="MR270">
 <attribute name="NAME" x="21.59" y="48.26" size="0.762" layer="22" font="vector" ratio="20" rot="MR0" align="center"/>
 <attribute name="PROD_ID" value=" " x="21.59" y="48.26" size="1.778" layer="28" rot="MR270" display="off"/>
 <attribute name="VALUE" x="22.733" y="48.26" size="0.6096" layer="28" font="vector" ratio="20" rot="MR270" align="top-center"/>
 </element>
-<element name="R11" library="SparkFun-Resistors" package="1206" value=" " x="12.7" y="39.37" smashed="yes" rot="R270">
+<element name="R11" library="SparkFun-Resistors" package="1206" value="470" x="12.7" y="39.37" smashed="yes" rot="R270">
 <attribute name="NAME" x="12.7" y="39.37" size="0.762" layer="21" font="vector" ratio="20" align="center"/>
 <attribute name="PROD_ID" value=" " x="12.7" y="39.37" size="1.778" layer="27" rot="R270" display="off"/>
 <attribute name="VALUE" x="11.557" y="39.37" size="0.6096" layer="27" font="vector" ratio="20" rot="R270" align="top-center"/>
 </element>
-<element name="R2" library="SparkFun-Resistors" package="1206" value=" " x="41.91" y="48.26" smashed="yes" rot="MR270">
+<element name="R2" library="SparkFun-Resistors" package="1206" value="470" x="41.91" y="48.26" smashed="yes" rot="MR270">
 <attribute name="NAME" x="41.91" y="48.26" size="0.762" layer="22" font="vector" ratio="20" rot="MR0" align="center"/>
 <attribute name="PROD_ID" value=" " x="41.91" y="48.26" size="1.778" layer="28" rot="MR270" display="off"/>
 <attribute name="VALUE" x="43.053" y="48.26" size="0.6096" layer="28" font="vector" ratio="20" rot="MR270" align="top-center"/>
 </element>
-<element name="R3" library="SparkFun-Resistors" package="1206" value=" " x="39.37" y="48.26" smashed="yes" rot="MR270">
+<element name="R3" library="SparkFun-Resistors" package="1206" value="470" x="39.37" y="48.26" smashed="yes" rot="MR270">
 <attribute name="NAME" x="39.37" y="48.26" size="0.762" layer="22" font="vector" ratio="20" rot="MR0" align="center"/>
 <attribute name="PROD_ID" value=" " x="39.37" y="48.26" size="1.778" layer="28" rot="MR270" display="off"/>
 <attribute name="VALUE" x="40.513" y="48.26" size="0.6096" layer="28" font="vector" ratio="20" rot="MR270" align="top-center"/>
 </element>
-<element name="R4" library="SparkFun-Resistors" package="1206" value=" " x="36.83" y="48.26" smashed="yes" rot="MR270">
+<element name="R4" library="SparkFun-Resistors" package="1206" value="470" x="36.83" y="48.26" smashed="yes" rot="MR270">
 <attribute name="NAME" x="36.83" y="48.26" size="0.762" layer="22" font="vector" ratio="20" rot="MR0" align="center"/>
 <attribute name="PROD_ID" value=" " x="36.83" y="48.26" size="1.778" layer="28" rot="MR270" display="off"/>
 <attribute name="VALUE" x="37.973" y="48.26" size="0.6096" layer="28" font="vector" ratio="20" rot="MR270" align="top-center"/>
 </element>
-<element name="R5" library="SparkFun-Resistors" package="1206" value=" " x="34.29" y="48.26" smashed="yes" rot="MR270">
+<element name="R5" library="SparkFun-Resistors" package="1206" value="470" x="34.29" y="48.26" smashed="yes" rot="MR270">
 <attribute name="NAME" x="34.29" y="48.26" size="0.762" layer="22" font="vector" ratio="20" rot="MR0" align="center"/>
 <attribute name="PROD_ID" value=" " x="34.29" y="48.26" size="1.778" layer="28" rot="MR270" display="off"/>
 <attribute name="VALUE" x="35.433" y="48.26" size="0.6096" layer="28" font="vector" ratio="20" rot="MR270" align="top-center"/>
 </element>
-<element name="R6" library="SparkFun-Resistors" package="1206" value=" " x="31.75" y="48.26" smashed="yes" rot="MR270">
+<element name="R6" library="SparkFun-Resistors" package="1206" value="470" x="31.75" y="48.26" smashed="yes" rot="MR270">
 <attribute name="NAME" x="31.75" y="48.26" size="0.762" layer="22" font="vector" ratio="20" rot="MR0" align="center"/>
 <attribute name="PROD_ID" value=" " x="31.75" y="48.26" size="1.778" layer="28" rot="MR270" display="off"/>
 <attribute name="VALUE" x="32.893" y="48.26" size="0.6096" layer="28" font="vector" ratio="20" rot="MR270" align="top-center"/>
 </element>
-<element name="R7" library="SparkFun-Resistors" package="1206" value=" " x="29.21" y="48.26" smashed="yes" rot="MR270">
+<element name="R7" library="SparkFun-Resistors" package="1206" value="470" x="29.21" y="48.26" smashed="yes" rot="MR270">
 <attribute name="NAME" x="29.21" y="48.26" size="0.762" layer="22" font="vector" ratio="20" rot="MR0" align="center"/>
 <attribute name="PROD_ID" value=" " x="29.21" y="48.26" size="1.778" layer="28" rot="MR270" display="off"/>
 <attribute name="VALUE" x="30.353" y="48.26" size="0.6096" layer="28" font="vector" ratio="20" rot="MR270" align="top-center"/>
 </element>
-<element name="R8" library="SparkFun-Resistors" package="1206" value=" " x="26.67" y="48.26" smashed="yes" rot="MR270">
+<element name="R8" library="SparkFun-Resistors" package="1206" value="470" x="26.67" y="48.26" smashed="yes" rot="MR270">
 <attribute name="NAME" x="26.67" y="48.26" size="0.762" layer="22" font="vector" ratio="20" rot="MR180" align="center"/>
 <attribute name="PROD_ID" value=" " x="26.67" y="48.26" size="1.778" layer="28" rot="MR270" display="off"/>
 <attribute name="VALUE" x="27.813" y="48.26" size="0.6096" layer="28" font="vector" ratio="20" rot="MR270" align="top-center"/>
 </element>
-<element name="R9" library="SparkFun-Resistors" package="1206" value=" " x="24.13" y="48.26" smashed="yes" rot="MR270">
+<element name="R9" library="SparkFun-Resistors" package="1206" value="470" x="24.13" y="48.26" smashed="yes" rot="MR270">
 <attribute name="NAME" x="24.13" y="48.26" size="0.762" layer="22" font="vector" ratio="20" rot="MR0" align="center"/>
 <attribute name="PROD_ID" value=" " x="24.13" y="48.26" size="1.778" layer="28" rot="MR270" display="off"/>
